File: YuSynthMiniMoog.kicad_sch (KiCad schematic)
At the start: 63 parts, among them J1 Conn_01x06_Socket, J2 Conn_01x03_Socket, J3 Conn_01x06_Socket, J4 Conn_01x02_Socket, J5 Conn_01x02_Socket, Q1 BC557, Q2 BC547, Q3 BC547, Q4 BC547, Q5 BC547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

Commit message: Add nonpolar caps
Parts:
- C10, C9: footprint (none) -> Capacitor_THT:C_Rect_L9.0mm_W2.5mm_P7.50mm_MKT; Manuf (none) -> Kemet; Manuf PN (none) -> C321C224K1R5TA
- C13: footprint (none) -> Capacitor_THT:C_Rect_L9.0mm_W2.5mm_P7.50mm_MKT; Manuf (none) -> Kemet; Manuf PN (none) -> C321C104Z5U5TA
- C14: footprint (none) -> Capacitor_THT:C_Rect_L4.0mm_W2.5mm_P2.50mm; Manuf (none) -> Kemet; Manuf PN (none) -> C315C101K5G5TA
- C4, C5, C6, C7: footprint (none) -> Capacitor_THT:C_Rect_L26.5mm_W8.5mm_P22.50mm_MKS4; Manuf (none) -> Kemet; Manuf PN (none) -> PHE426DJ5470JR05
Changed lines of the file:
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@@
       (effects (font (size 1.27 1.27)))
     )
-    (property "Footprint" "" (at 229.87 75.2348 0)
+    (property "Footprint" "Capacitor_THT:C_Rect_L9.0mm_W2.5mm_P7.50mm_MKT" (at 229.87 75.2348 0)
       (effects (font (size 1.27 1.27)) hide)
     )
     (property "Datasheet" "~" (at 226.06 76.2 0)
+      (effects (font (size 1.27 1.27)) hide)
+    )
+    (property "Manuf" "Kemet" (at 226.06 76.2 90)
+      (effects (font (size 1.27 1.27)) hide)
+    )
+    (property "Manuf PN" "C321C224K1R5TA" (at 226.06 76.2 90)
       (effects (font (size 1.27 1.27)) hide)
     )
@@
       (effects (font (size 1.27 1.27)))
     )
-    (property "Footprint" "" (at 193.04 81.5848 0)
-      (effects (font (size 1.27 1.27)) hide)
-    )
-    (property "Datasheet" "~" (at 189.23 82.55 0)
+    (property "Footprint" "Capacitor_THT:C_Rect_L26.5mm_W8.5mm_P22.50mm_MKS4" (at 193.04 81.5848 0)
+      (effects (font (size 1.27 1.27)) hide)
+    )
+    (property "Datasheet" "https://connect.kemet.com:7667/gateway/IntelliData-ComponentDocumentation/1.0/download/datasheet/PHE426DJ5470JR05" (at 189.23 82.55 0)
+      (effects (font (size 1.27 1.27)) hide)
+    )
+    (property "Manuf" "Kemet" (at 189.23 82.55 90)
+      (effects (font (size 1.27 1.27)) hide)
+    )
+    (property "Manuf PN" "PHE426DJ5470JR05" (at 189.23 82.55 90)
       (effects (font (size 1.27 1.27)) hide)
     )
@@
       (effects (font (size 1.27 1.27)))
     )
-    (property "Footprint" "" (at 193.04 132.3848 0)
-      (effects (font (size 1.27 1.27)) hide)
-    )
-    (property "Datasheet" "~" (at 189.23 133.35 0)
+    (property "Footprint" "Capacitor_THT:C_Rect_L26.5mm_W8.5mm_P22.50mm_MKS4" (at 193.04 132.3848 0)
+      (effects (font (size 1.27 1.27)) hide)
+    )
+    (property "Datasheet" "https://connect.kemet.com:7667/gateway/IntelliData-ComponentDocumentation/1.0/download/datasheet/PHE426DJ5470JR05" (at 189.23 133.35 0)
+      (effects (font (size 1.27 1.27)) hide)
+    )
+    (property "Manuf" "Kemet" (at 189.23 133.35 90)
+      (effects (font (size 1.27 1.27)) hide)
+    )
+    (property "Manuf PN" "PHE426DJ5470JR05" (at 189.23 133.35 90)
       (effects (font (size 1.27 1.27)) hide)
     )
@@
       (effects (font (size 1.27 1.27)))
     )
-    (property "Footprint" "" (at 193.04 98.0948 0)
-      (effects (font (size 1.27 1.27)) hide)
-    )
-    (property "Datasheet" "~" (at 189.23 99.06 0)
+    (property "Footprint" "Capacitor_THT:C_Rect_L26.5mm_W8.5mm_P22.50mm_MKS4" (at 193.04 98.0948 0)
+      (effects (font (size 1.27 1.27)) hide)
+    )
+    (property "Datasheet" "https://connect.kemet.com:7667/gateway/IntelliData-ComponentDocumentation/1.0/download/datasheet/PHE426DJ5470JR05" (at 189.23 99.06 0)
+      (effects (font (size 1.27 1.27)) hide)
+    )
+    (property "Manuf" "Kemet" (at 189.23 99.06 90)
+      (effects (font (size 1.27 1.27)) hide)
+    )
+    (property "Manuf PN" "PHE426DJ5470JR05" (at 189.23 99.06 90)
       (effects (font (size 1.27 1.27)) hide)
     )
@@
       (effects (font (size 1.27 1.27)))
     )
-    (property "Footprint" "" (at 193.04 114.6048 0)
-      (effects (font (size 1.27 1.27)) hide)
-    )
-    (property "Datasheet" "~" (at 189.23 115.57 0)
+    (property "Footprint" "Capacitor_THT:C_Rect_L26.5mm_W8.5mm_P22.50mm_MKS4" (at 193.04 114.6048 0)
+      (effects (font (size 1.27 1.27)) hide)
+    )
+    (property "Datasheet" "https://connect.kemet.com:7667/gateway/IntelliData-ComponentDocumentation/1.0/download/datasheet/PHE426DJ5470JR05" (at 189.23 115.57 0)
+      (effects (font (size 1.27 1.27)) hide)
+    )
+    (property "Manuf" "Kemet" (at 189.23 115.57 90)
+      (effects (font (size 1.27 1.27)) hide)
+    )
+    (property "Manuf PN" "PHE426DJ5470JR05" (at 189.23 115.57 90)
       (effects (font (size 1.27 1.27)) hide)
     )
@@
       (effects (font (size 1.27 1.27)) (justify left))
     )
-    (property "Footprint" "" (at 121.6152 95.25 0)
+    (property "Footprint" "Capacitor_THT:C_Rect_L9.0mm_W2.5mm_P7.50mm_MKT" (at 121.6152 95.25 0)
       (effects (font (size 1.27 1.27)) hide)
     )
     (property "Datasheet" "~" (at 120.65 91.44 0)
+      (effects (font (size 1.27 1.27)) hide)
+    )
+    (property "Manuf" "Kemet" (at 120.65 91.44 0)
+      (effects (font (size 1.27 1.27)) hide)
+    )
+    (property "Manuf PN" "C321C104Z5U5TA" (at 120.65 91.44 0)
       (effects (font (size 1.27 1.27)) hide)
     )
@@
       (effects (font (size 1.27 1.27)) (justify left))
     )
-    (property "Footprint" "" (at 127.9652 210.82 0)
+    (property "Footprint" "Capacitor_THT:C_Rect_L4.0mm_W2.5mm_P2.50mm" (at 127.9652 210.82 0)
       (effects (font (size 1.27 1.27)) hide)
     )
     (property "Datasheet" "~" (at 127 207.01 0)
+      (effects (font (size 1.27 1.27)) hide)
+    )
+    (property "Manuf" "Kemet" (at 127 207.01 0)
+      (effects (font (size 1.27 1.27)) hide)
+    )
+    (property "Manuf PN" "C315C101K5G5TA" (at 127 207.01 0)
       (effects (font (size 1.27 1.27)) hide)
     )
@@
       (effects (font (size 1.27 1.27)))
     )
-    (property "Footprint" "" (at 224.79 79.0448 0)
+    (property "Footprint" "Capacitor_THT:C_Rect_L9.0mm_W2.5mm_P7.50mm_MKT" (at 224.79 79.0448 0)
       (effects (font (size 1.27 1.27)) hide)
     )
@@
       (effects (font (size 1.27 1.27)) hide)
     )
+    (property "Manuf" "Kemet" (at 220.98 80.01 90)
+      (effects (font (size 1.27 1.27)) hide)
+    )
+    (property "Manuf PN" "C321C224K1R5TA" (at 220.98 80.01 90)
+      (effects (font (size 1.27 1.27)) hide)
+    )
